File: interzone.kicad_pcb (KiCad board)
At the start: 2 copper layers, 265.3 x 128.5 mm, 58 parts, among them J101 Barrel_Jack_Switch_Pin3Ring, J102 Barrel_Jack_Switch_Pin3Ring, J103 Barrel_Jack_Switch_Pin3Ring, J104 Barrel_Jack_Switch_Pin3Ring, J105 Barrel_Jack_Switch_Pin3Ring, J106 Barrel_Jack_Switch_Pin3Ring, J107 Barrel_Jack_Switch_Pin3Ring, J108 Barrel_Jack_Switch_Pin3Ring, J109 Conn_01x16, J110 Conn_02x16_Odd_Even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

Commit message: remove jack footprints from faceplate
Parts:
- removed the J101 at (67.5, 49.5)
- removed the J102 at (81.9, 49.5)
- removed the J103 at (96.3, 49.5)
- removed the J104 at (110.7, 49.5)
Changed lines of the file:
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@@
       (thermal_bridge_angle 45))
-  )
-  (footprint "interzone:XKC PJ-3411" (layer "F.Cu")
-    (at 96.266532 49.499475 180)
-    (property "Sheetfile" "interzone.kicad_sch")
-    (property "Sheetname" "")
-    (property "ki_description" "DC Barrel Jack with an internal switch")
-    (property "ki_keywords" "DC power barrel jack connector")
-    (attr smd)
-    (fp_text reference "J103" (at 0 -8 180 unlocked) (layer "F.SilkS") hide
-        (effects (font (size 1 1) (thickness 0.1)))
-    )
-    (fp_text value "Barrel_Jack_Switch_Pin3Ring" (at 0 1 180 unlocked) (layer "F.Fab")
-        (effects (font (size 1 1) (thickness 0.15)))
-    )
-    (fp_text user "${REFERENCE}" (at 0 2.5 180 unlocked) (layer "F.Fab")
-        (effects (font (size 1 1) (thickness 0.15)))
-    )
-    (fp_line (start -5.5 -5) (end -2 -5)
-      (stroke (width 0.1) (type default)) (layer "F.SilkS"))
-    (fp_line (start -5.5 5) (end -5.5 -5)
-      (stroke (width 0.1) (type default)) (layer "F.SilkS"))
-    (fp_line (start -5.5 5) (end -2 5)
-      (stroke (width 0.1) (type default)) (layer "F.SilkS"))
-    (fp_line (start 5.75 -5) (end 2 -5)
-      (stroke (width 0.1) (type default)) (layer "F.SilkS"))
-    (fp_line (start 5.75 -5) (end 5.75 -1.75)
-      (stroke (width 0.1) (type default)) (layer "F.SilkS"))
-    (fp_line (start 5.75 1.75) (end 5.75 5)
-      (stroke (width 0.1) (type default)) (layer "F.SilkS"))
-    (fp_line (start 5.75 5) (end 2 5)
-      (stroke (width 0.1) (type default)) (layer "F.SilkS"))
-    (fp_arc (start 4.949747 2.12132) (mid -5.384764 -0.065658) (end 4.999999 -2)
-      (stroke (width 0.1) (type default)) (layer "F.SilkS"))
-    (pad "R" thru_hole oval (at -3.2 0) (size 1.5 3.1) (drill oval 0.9 2.5) (layers "*.Cu" "*.Mask")
-      (net 14 "Net-(J116-Pin_10)") (pintype "passive") (thermal_bridge_angle 45))
-    (pad "S" thru_hole oval (at 0 -3.5 270) (size 1.5 3.1) (drill oval 0.9 2.5) (layers "*.Cu" "*.Mask")
-      (net 1 "GND") (pinfunction "S") (pintype "passive") (thermal_bridge_angle 45))
-    (pad "T" thru_hole oval (at 5.141 0) (size 1.5 3.1) (drill oval 0.9 2.5) (layers "*.Cu" "*.Mask")
-      (net 15 "Net-(J112-Pin_10)") (pintype "passive") (thermal_bridge_angle 45))
   )
   (footprint "interzone:XKC PJ-3411-hole" (layer "F.Cu")
@@
       (net 15 "Net-(J112-Pin_10)") (pintype "passive") (thermal_bridge_angle 45))
   )
-  (footprint "interzone:XKC PJ-3411" (layer "F.Cu")
-    (at 81.864866 49.499475 180)
-    (property "Sheetfile" "interzone.kicad_sch")
-    (property "Sheetname" "")
-    (property "ki_description" "DC Barrel Jack with an internal switch")
-    (property "ki_keywords" "DC power barrel jack connector")
-    (attr smd)
-    (fp_text reference "J102" (at 0 -8 180 unlocked) (layer "F.SilkS") hide
-        (effects (font (size 1 1) (thickness 0.1)))
-    )
-    (fp_text value "Barrel_Jack_Switch_Pin3Ring" (at 0 1 180 unlocked) (layer "F.Fab")
-        (effects (font (size 1 1) (thickness 0.15)))
-    )
-    (fp_text user "${REFERENCE}" (at 0 2.5 180 unlocked) (layer "F.Fab")
-        (effects (font (size 1 1) (thickness 0.15)))
-    )
-    (fp_line (start -5.5 -5) (end -2 -5)
-      (stroke (width 0.1) (type default)) (layer "F.SilkS"))
-    (fp_line (start -5.5 5) (end -5.5 -5)
-      (stroke (width 0.1) (type default)) (layer "F.SilkS"))
-    (fp_line (start -5.5 5) (end -2 5)
-      (stroke (width 0.1) (type default)) (layer "F.SilkS"))
-    (fp_line (start 5.75 -5) (end 2 -5)
-      (stroke (width 0.1) (type default)) (layer "F.SilkS"))
-    (fp_line (start 5.75 -5) (end 5.75 -1.75)
-      (stroke (width 0.1) (type default)) (layer "F.SilkS"))
-    (fp_line (start 5.75 1.75) (end 5.75 5)
-      (stroke (width 0.1) (type default)) (layer "F.SilkS"))
-    (fp_line (start 5.75 5) (end 2 5)
-      (stroke (width 0.1) (type default)) (layer "F.SilkS"))
-    (fp_arc (start 4.949747 2.12132) (mid -5.384764 -0.065658) (end 4.999999 -2)
-      (stroke (width 0.1) (type default)) (layer "F.SilkS"))
-    (pad "R" thru_hole oval (at -3.2 0) (size 1.5 3.1) (drill oval 0.9 2.5) (layers "*.Cu" "*.Mask")
-      (net 12 "Net-(J115-Pin_10)") (pintype "passive") (thermal_bridge_angle 45))
-    (pad "S" thru_hole oval (at 0 -3.5 270) (size 1.5 3.1) (drill oval 0.9 2.5) (layers "*.Cu" "*.Mask")
-      (net 1 "GND") (pinfunction "S") (pintype "passive") (thermal_bridge_angle 45))
-    (pad "T" thru_hole oval (at 5.141 0) (size 1.5 3.1) (drill oval 0.9 2.5) (layers "*.Cu" "*.Mask")
-      (net 13 "Net-(J111-Pin_10)") (pintype "passive") (thermal_bridge_angle 45))
-  )
-  (footprint "interzone:XKC PJ-3411" (layer "F.Cu")
-    (at 67.4632 49.499475 180)
-    (property "Sheetfile" "interzone.kicad_sch")
-    (property "Sheetname" "")
-    (property "ki_description" "DC Barrel Jack with an internal switch")
-    (property "ki_keywords" "DC power barrel jack connector")
-    (attr smd)
-    (fp_text reference "J101" (at 0 -8 180 unlocked) (layer "F.SilkS")
-        (effects (font (size 1 1) (thickness 0.1)))
-    )
-    (fp_text value "Barrel_Jack_Switch_Pin3Ring" (at 0 1 180 unlocked) (layer "F.Fab")
-        (effects (font (size 1 1) (thickness 0.15)))
-    )
-    (fp_text user "${REFERENCE}" (at 0 2.5 180 unlocked) (layer "F.Fab")
-        (effects (font (size 1 1) (thickness 0.15)))
-    )
-    (fp_line (start -5.5 -5) (end -2 -5)
-      (stroke (width 0.1) (type default)) (layer "F.SilkS"))
-    (fp_line (start -5.5 5) (end -5.5 -5)
-      (stroke (width 0.1) (type default)) (layer "F.SilkS"))
-    (fp_line (start -5.5 5) (end -2 5)
-      (stroke (width 0.1) (type default)) (layer "F.SilkS"))
-    (fp_line (start 5.75 -5) (end 2 -5)
-      (stroke (width 0.1) (type default)) (layer "F.SilkS"))
-    (fp_line (start 5.75 -5) (end 5.75 -1.75)
-      (stroke (width 0.1) (type default)) (layer "F.SilkS"))
-    (fp_line (start 5.75 1.75) (end 5.75 5)
-      (stroke (width 0.1) (type default)) (layer "F.SilkS"))
-    (fp_line (start 5.75 5) (end 2 5)
-      (stroke (width 0.1) (type default)) (layer "F.SilkS"))
-    (fp_arc (start 4.949747 2.12132) (mid -5.384764 -0.065658) (end 4.999999 -2)
-      (stroke (width 0.1) (type default)) (layer "F.SilkS"))
-    (pad "R" thru_hole oval (at -3.2 0) (size 1.5 3.1) (drill oval 0.9 2.5) (layers "*.Cu" "*.Mask")
-      (net 10 "Net-(J114-Pin_10)") (pintype "passive") (thermal_bridge_angle 45))
-    (pad "S" thru_hole oval (at 0 -3.5 270) (size 1.5 3.1) (drill oval 0.9 2.5) (layers "*.Cu" "*.Mask")
-      (net 1 "GND") (pinfunction "S") (pintype "passive") (thermal_bridge_angle 45))
-    (pad "T" thru_hole oval (at 5.141 0) (size 1.5 3.1) (drill oval 0.9 2.5) (layers "*.Cu" "*.Mask")
-      (net 11 "Net-(J110-Pin_10)") (pintype "passive") (thermal_bridge_angle 45))
-  )
   (footprint "Connector_PinSocket_2.54mm:PinSocket_2x16_P2.54mm_Vertical" (layer "F.Cu")
     (at 207.19 71.64)
@@
     )
   )
-  (footprint "interzone:XKC PJ-3411" (layer "F.Cu")
-    (at 110.6682 49.499475 180)
-    (property "Sheetfile" "interzone.kicad_sch")
-    (property "Sheetname" "")
-    (property "ki_description" "DC Barrel Jack with an internal switch")
-    (property "ki_keywords" "DC power barrel jack connector")
-    (attr smd)
-    (fp_text reference "J104" (at 0 -8 180 unlocked) (layer "F.SilkS") hide
-        (effects (font (size 1 1) (thickness 0.1)))
-    )
-    (fp_text value "Barrel_Jack_Switch_Pin3Ring" (at 0 1 180 unlocked) (layer "F.Fab")
-        (effects (font (size 1 1) (thickness 0.15)))
-    )
-    (fp_text user "${REFERENCE}" (at 0 2.5 180 unlocked) (layer "F.Fab")
-        (effects (font (size 1 1) (thickness 0.15)))
-    )
-    (fp_line (start -5.5 -5) (end -2 -5)
-      (stroke (width 0.1) (type default)) (layer "F.SilkS"))
-    (fp_line (start -5.5 5) (end -5.5 -5)
-      (stroke (width 0.1) (type default)) (layer "F.SilkS"))
-    (fp_line (start -5.5 5) (end -2 5)
-      (stroke (width 0.1) (type default)) (layer "F.SilkS"))
-    (fp_line (start 5.75 -5) (end 2 -5)
-      (stroke (width 0.1) (type default)) (layer "F.SilkS"))
-    (fp_line (start 5.75 -5) (end 5.75 -1.75)
-      (stroke (width 0.1) (type default)) (layer "F.SilkS"))
-    (fp_line (start 5.75 1.75) (end 5.75 5)
-      (stroke (width 0.1) (type default)) (layer "F.SilkS"))
-    (fp_line (start 5.75 5) (end 2 5)
-      (stroke (width 0.1) (type default)) (layer "F.SilkS"))
-    (fp_arc (start 4.949747 2.12132) (mid -5.384764 -0.065658) (end 4.999999 -2)
-      (stroke (width 0.1) (type default)) (layer "F.SilkS"))
-    (pad "R" thru_hole oval (at -3.2 0) (size 1.5 3.1) (drill oval 0.9 2.5) (layers "*.Cu" "*.Mask")
-      (net 16 "Net-(J117-Pin_10)") (pintype "passive") (thermal_bridge_angle 45))
-    (pad "S" thru_hole oval (at 0 -3.5 270) (size 1.5 3.1) (drill oval 0.9 2.5) (layers "*.Cu" "*.Mask")
-      (net 1 "GND") (pinfunction "S") (pintype "passive") (thermal_bridge_angle 45))
-    (pad "T" thru_hole oval (at 5.141 0) (size 1.5 3.1) (drill oval 0.9 2.5) (layers "*.Cu" "*.Mask")
-      (net 17 "Net-(J113-Pin_10)") (pintype "passive") (thermal_bridge_angle 45))
-  )
   (footprint "Connector_PinHeader_2.54mm:PinHeader_1x16_P2.54mm_Vertical" (layer "F.Cu")

Commit message: added grant edits
Other:
- board text added: "A"
- board text added: "ASSOCIATES"
- board text added: "B"
- board text added: "GND"
- board text added: "I/O BANK A"
- board text added: "I/O BANK B"
- board text added: "Interzone"
- board text added: "R1"
- board text added: "R2"
- board text added: "R3"
- board text added: "R4"
- board text added: "T1"
- board text added: "T2"
- board text added: "T3"
- board text added: "T4"
- board text added: "{dblquote}It is the zone between the real world and the imagination, Bill.{dblquote}"
